File: Ejercicio2/Conector.sch (KiCad schematic (older format))
At the start: 1 part

Commit message: Agrego bus al esquemático. Quito resistor adicional.
Parts:
- XA1: footprint (none) -> ej2:Conn_Poncho_Derecha
Other:
- note added: "Etiqueta \nglobal"
- note added: "Etiquetas\nde Jerarquía"
- note added: "Power\nFlag"
Changed lines of the file:
@@
 EESchema Schematic File Version 2
-LIBS:sp3232e
-LIBS:c
-LIBS:power
-LIBS:device
+LIBS:ej2
 LIBS:ej2-cache
 EELAYER 25 0
@@
 F 0 "XA1" H 5600 3350 60  0000 C CNN
 F 1 "Conn_Poncho2P_2x_20x2" H 5650 1250 60  0000 C CNN
-F 2 "" H 5300 2950 60  0000 C CNN
+F 2 "ej2:Conn_Poncho_Derecha" H 5300 2950 60  0001 C CNN
 F 3 "" H 5300 2950 60  0000 C CNN
 	1    5300 2950
@@
 $EndComp
 Connection ~ 6650 2750
+Wire Notes Line
+	4750 2400 4600 2250
+Wire Notes Line
+	4600 2250 4400 2250
+Wire Notes Line
+	4000 3650 3900 3650
+Wire Notes Line
+	3900 3650 3900 4600
+Wire Notes Line
+	3900 4600 4000 4600
+Text Notes 3250 3950 0    60   ~ 0
+Etiquetas\nde Jerarquía
+Text Notes 4050 2200 0    60   ~ 0
+Etiqueta \nglobal
+Wire Notes Line
+	6850 2500 6950 2400
+Wire Notes Line
+	6950 2400 7150 2400
+Text Notes 7200 2450 0    60   ~ 0
+Power\nFlag
 $EndSCHEMATC

Commit message: Cambio numeración (OJO:PCB ROTO), cambio plugin BOM, quito R de VCC.
Parts:
- XA1: Digikey/Mouser (none) -> 952-1387-ND
Changed lines of the file:
@@
 EESchema Schematic File Version 2
 LIBS:ej2
+LIBS:power
 LIBS:ej2-cache
 EELAYER 25 0
@@
 F 1 "Conn_Poncho2P_2x_20x2" H 5650 1250 60  0000 C CNN
 F 2 "ej2:Conn_Poncho_Derecha" H 5300 2950 60  0001 C CNN
-F 3 "" H 5300 2950 60  0000 C CNN
+F 3 "https://cdn.harwin.com/pdfs/60page108.pdf" H 5300 2950 60  0001 C CNN
+F 4 "952-1387-ND" H 5300 2950 60  0001 C CNN "Digikey/Mouser"
 	1    5300 2950
 	1    0    0    -1
 $EndComp
 $Comp
-L +3.3V #PWR01
+L +3.3V #PWR1
 U 1 1 564E1CF0
 P 4850 2550
-F 0 "#PWR01" H 4850 2510 30  0001 C CNN
+F 0 "#PWR1" H 4850 2510 30  0001 C CNN
 F 1 "+3.3V" H 4850 2660 30  0000 C CNN
 F 2 "" H 4850 2550 60  0000 C CNN
@@
 $EndComp
 $Comp
-L GND #PWR02
+L GND #PWR2
 U 1 1 564E1D0B
 P 6650 4700
-F 0 "#PWR02" H 6650 4700 30  0001 C CNN
+F 0 "#PWR2" H 6650 4700 30  0001 C CNN
 F 1 "GND" H 6650 4630 30  0001 C CNN
 F 2 "" H 6650 4700 60  0000 C CNN
@@
 NoConn ~ 5050 4550
 $Comp
-L PWR_FLAG #FLG03
+L PWR_FLAG #FLG1
 U 1 1 564F7667
 P 6650 2700
-F 0 "#FLG03" H 6650 2795 30  0001 C CNN
+F 0 "#FLG1" H 6650 2795 30  0001 C CNN
 F 1 "PWR_FLAG" H 6650 2880 30  0000 C CNN
 F 2 "" H 6650 2700 60  0000 C CNN

Commit message: Versión del Ejercicio2 con CAN.
Parts:
- added C6: 100nF, Capacitors_SMD:C_1206_HandSoldering, symbol C
- added J2: CAN, ej2:CON_PALETA_3, symbol CONN_3
- added R1, R2: 60, Resistors_SMD:R_1206_HandSoldering, symbol R
- added U2: AMIS42665TJAA1RG, ej2:SOIC-8, symbol AMIS42665TJAA1RG
Connections:
- net GND: now also C6.1, J2.3, U2.2 (GND), U2.8 (STB)
- net +5V: now reaches XA1.2 (+5V)
- net +5V: now also C6.2, U2.3 (VCC)
- net CAN_RX: now reaches XA1.27 (canRD)
- net CAN_RX: now also U2.4 (RXD)
- net CAN_TX: now reaches XA1.29 (canTD)
- net CAN_TX: now also U2.1 (TXD)
- new net: R1.2, R2.1, U2.5 (SPLIT)
- new net CAN_N: J2.2, R2.2, U2.6 (CANL)
- new net CAN_P: J2.1, R1.1, U2.7 (CANH)
- no-connect marks 25 -> 22
Other:
- note added: "Etiquetas\nlocales"
- note added: "Par diferencial\n120 Ohms"
Changed lines of the file:
@@
 LIBS:ej2
 LIBS:power
-LIBS:ej2-cache
 EELAYER 25 0
 EELAYER END
@@
 encoding utf-8
 Sheet 2 3
-Title "Ejercicio 2 - Curso Kicad"
-Date "2015-11-19"
+Title "Ejercicio 2 - Curso Kicad - Hoja Conector y CAN"
+Date "2015-11-26"
 Rev "1.0"
 Comp "Instituto Nacional de Tecnología Industrial INTI-CMNB"
-Comment1 ""
+Comment1 "Autores: D. Alamon, D. Brengi, N. Scotti"
 Comment2 ""
 Comment3 ""
@@
 $EndComp
 $Comp
-L +3.3V #PWR1
+L +3.3V #PWR01
 U 1 1 564E1CF0
 P 4850 2550
-F 0 "#PWR1" H 4850 2510 30  0001 C CNN
+F 0 "#PWR01" H 4850 2510 30  0001 C CNN
 F 1 "+3.3V" H 4850 2660 30  0000 C CNN
 F 2 "" H 4850 2550 60  0000 C CNN
@@
 $EndComp
 $Comp
-L GND #PWR2
+L GND #PWR02
 U 1 1 564E1D0B
 P 6650 4700
-F 0 "#PWR2" H 6650 4700 30  0001 C CNN
+F 0 "#PWR02" H 6650 4700 30  0001 C CNN
 F 1 "GND" H 6650 4630 30  0001 C CNN
 F 2 "" H 6650 4700 60  0000 C CNN
@@
 NoConn ~ 6250 2950
 NoConn ~ 6250 2850
-NoConn ~ 6250 2650
 NoConn ~ 5050 2750
 NoConn ~ 5050 2850
@@
 NoConn ~ 5050 3550
 NoConn ~ 5050 3650
-NoConn ~ 5050 3950
-NoConn ~ 5050 4050
 NoConn ~ 5050 4150
 NoConn ~ 5050 4250
 NoConn ~ 5050 4550
 $Comp
-L PWR_FLAG #FLG1
+L PWR_FLAG #FLG03
 U 1 1 564F7667
 P 6650 2700
-F 0 "#FLG1" H 6650 2795 30  0001 C CNN
+F 0 "#FLG03" H 6650 2795 30  0001 C CNN
 F 1 "PWR_FLAG" H 6650 2880 30  0000 C CNN
 F 2 "" H 6650 2700 60  0000 C CNN
@@
 Text Notes 7200 2450 0    60   ~ 0
 Power\nFlag
+$Comp
+L CONN_3 J2
+U 1 1 56563B7F
+P 7450 3750
+F 0 "J2" H 7500 3750 60  0000 C CNN
+F 1 "CAN" H 7500 3250 60  0000 C CNN
+F 2 "ej2:CON_PALETA_3" H 7450 3750 60  0001 C CNN
+F 3 "" H 7450 3750 60  0000 C CNN
+	1    7450 3750
+	-1   0    0    -1
+$EndComp
+$Comp
+L AMIS42665TJAA1RG U2
+U 1 1 565737A4
+P 9050 4000
+F 0 "U2" H 9350 4500 60  0000 C CNN
+F 1 "AMIS42665TJAA1RG" H 9050 3600 60  0000 C CNN
+F 2 "ej2:SOIC-8" H 9050 4050 60  0001 C CNN
+F 3 "" H 9050 4050 60  0000 C CNN
+	1    9050 4000
+	-1   0    0    -1
+$EndComp
+$Comp
+L +5V #PWR04
+U 1 1 5657394E
+P 6400 2550
+F 0 "#PWR04" H 6400 2400 50  0001 C CNN
+F 1 "+5V" H 6400 2690 30  0000 C CNN
+F 2 "" H 6400 2550 60  0000 C CNN
+F 3 "" H 6400 2550 60  0000 C CNN
+	1    6400 2550
+	1    0    0    -1
+$EndComp
+Wire Wire Line
+	6250 2650 6400 2650
+Wire Wire Line
+	6400 2650 6400 2550
+$Comp
+L +5V #PWR05
+U 1 1 565739CF
+P 9700 3600
+F 0 "#PWR05" H 9700 3450 50  0001 C CNN
+F 1 "+5V" H 9700 3740 30  0000 C CNN
+F 2 "" H 9700 3600 60  0000 C CNN
+F 3 "" H 9700 3600 60  0000 C CNN
+	1    9700 3600
+	1    0    0    -1
+$EndComp
+$Comp
+L C C6
+U 1 1 56573B2C
+P 9950 3650
+F 0 "C6" V 9800 3750 40  0000 L CNN
+F 1 "100nF" V 9900 3750 40  0000 L CNN
+F 2 "Capacitors_SMD:C_1206_HandSoldering" H 9988 3500 30  0001 C CNN
+F 3 "http://www.yageo.com/documents/recent/UPY-GPHC_X7R_6.3V-to-50V-v12.pdf" H 9950 3650 60  0001 C CNN
+F 4 "311-1179-1-ND" H 9950 3650 60  0001 C CNN "Digikey/Mouser"
+	1    9950 3650
+	0    1    1    0
+$EndComp
+$Comp
+L R R1
+U 1 1 5657407D
+P 8150 3650
+F 0 "R1" V 8050 3650 50  0000 C CNN
+F 1 "60" V 8150 3650 50  0000 C CNN
+F 2 "Resistors_SMD:R_1206_HandSoldering" H 8150 3650 60  0001 C CNN
+F 3 "" H 8150 3650 60  0000 C CNN
+	1    8150 3650
+	1    0    0    -1
+$EndComp
+$Comp
+L R R2
+U 1 1 565744AF
+P 8150 4250
+F 0 "R2" V 8050 4250 50  0000 C CNN
+F 1 "60" V 8150 4250 50  0000 C CNN
+F 2 "Resistors_SMD:R_1206_HandSoldering" H 8150 4250 60  0001 C CNN
+F 3 "" H 8150 4250 60  0000 C CNN
+	1    8150 4250
+	1    0    0    -1
+$EndComp
+Text Label 4950 4050 2    60   ~ 0
+CAN_TX
+Text Label 4950 3950 2    60   ~ 0
+CAN_RX
+Text Label 9800 3950 0    60   ~ 0
+CAN_TX
+Wire Notes Line
+	4850 4100 4850 5050
+Wire Notes Line
+	4850 5050 5300 5050
+Text Notes 5350 5150 0    60   ~ 0
+Etiquetas\nlocales
+Text Label 9800 4100 0    60   ~ 0
+CAN_RX
+$Comp
+L GND #PWR06
+U 1 1 56574828
+P 9750 4350
+F 0 "#PWR06" H 9750 4350 30  0001 C CNN
+F 1 "GND" H 9750 4280 30  0001 C CNN
+F 2 "" H 9750 4350 60  0000 C CNN
+F 3 "" H 9750 4350 60  0000 C CNN
+	1    9750 4350
+	1    0    0    -1
+$EndComp
+Wire Wire Line
+	5050 3950 4950 3950
+Wire Wire Line
+	5050 4050 4950 4050
+Wire Wire Line
+	9650 3950 9800 3950
+Wire Wire Line
+	9650 4100 9800 4100
+Wire Wire Line
+	9650 3800 9750 3800
+Wire Wire Line
+	9750 3800 9750 4350
+Wire Wire Line
+	9650 4250 9750 4250
+Connection ~ 9750 4250
+$Comp
+L GND #PWR07
+U 1 1 56574BF8
+P 10200 3700
+F 0 "#PWR07" H 10200 3700 30  0001 C CNN
+F 1 "GND" H 10200 3630 30  0001 C CNN
+F 2 "" H 10200 3700 60  0000 C CNN
+F 3 "" H 10200 3700 60  0000 C CNN
+	1    10200 3700
+	1    0    0    -1
+$EndComp
+Wire Wire Line
+	10150 3650 10200 3650
+Wire Wire Line
+	9650 3650 9750 3650
+Wire Wire Line
+	9700 3600 9700 3650
+Connection ~ 9700 3650
+$Comp
+L GND #PWR08
+U 1 1 56574E5F
+P 7700 4150
+F 0 "#PWR08" H 7700 4150 30  0001 C CNN
+F 1 "GND" H 7700 4080 30  0001 C CNN
+F 2 "" H 7700 4150 60  0000 C CNN
+F 3 "" H 7700 4150 60  0000 C CNN
+	1    7700 4150
+	1    0    0    -1
+$EndComp
+Wire Wire Line
+	7650 4100 7700 4100
+Wire Wire Line
+	7700 4100 7700 4150
+Wire Wire Line
+	8350 3350 8350 3650
+Wire Wire Line
+	8350 3650 8400 3650
+Wire Wire Line
+	8150 3400 8150 3350
+Connection ~ 8150 3350
+Wire Wire Line
+	8400 4250 8350 4250
+Wire Wire Line
+	8350 4250 8350 4550
+Wire Wire Line
+	8350 4550 7950 4550
+Wire Wire Line
+	7950 4550 7950 4000
+Wire Wire Line
+	7950 4000 7650 4000
+Wire Wire Line
+	8350 3350 7950 3350
+Wire Wire Line
+	7950 3350 7950 3900
+Wire Wire Line
+	7950 3900 7650 3900
+Wire Notes Line
+	7850 4100 7850 4800
+Wire Notes Line
+	7850 4800 8100 4800
+Text Notes 8150 4900 0    60   ~ 0
+Par diferencial\n120 Ohms
+Text Label 7650 3900 0    60   ~ 0
+CAN_P
+Text Label 7650 4000 0    60   ~ 0
+CAN_N
+Wire Wire Line
+	8150 3900 8150 4000
+Wire Wire Line
+	8150 3950 8400 3950
+Connection ~ 8150 3950
+Wire Wire Line
+	8150 4500 8150 4550
+Connection ~ 8150 4550
+Wire Wire Line
+	10200 3650 10200 3700
 $EndSCHEMATC
