File: Ejercicio2/Conector.sch (KiCad schematic (older format))
At the start: 6 parts, among them J2 CAN, U2 AMIS42665TJAA1RG

Commit message: Completos campos en el esquemático.
Parts:
- J2: Digikey/Mouser (none) -> A19470-ND
- R1, R2: Digikey/Mouser (none) -> Y149660R0000A0R-ND
- U2: Digikey/Mouser (none) -> 766-1006-1-ND
Changed lines of the file:
@@
 F 1 "CAN" H 7500 3250 60  0000 C CNN
 F 2 "ej2:CON_PALETA_3" H 7450 3750 60  0001 C CNN
-F 3 "" H 7450 3750 60  0000 C CNN
+F 3 "http://www.te.com/commerce/DocumentDelivery/DDEController?Action=srchrtrv&DocNm=640456&DocType=Customer+Drawing&DocLang=English" H 7450 3750 60  0001 C CNN
+F 4 "A19470-ND" H 7450 3750 60  0001 C CNN "Digikey/Mouser"
 	1    7450 3750
 	-1   0    0    -1
@@
 F 1 "AMIS42665TJAA1RG" H 9050 3600 60  0000 C CNN
 F 2 "ej2:SOIC-8" H 9050 4050 60  0001 C CNN
-F 3 "" H 9050 4050 60  0000 C CNN
+F 3 "http://www.onsemi.com/pub_link/Collateral/AMIS-42665-D.PDF" H 9050 4050 60  0001 C CNN
+F 4 "766-1006-1-ND" H 9050 4000 60  0001 C CNN "Digikey/Mouser"
 	1    9050 4000
 	-1   0    0    -1
@@
 F 1 "60" V 8150 3650 50  0000 C CNN
 F 2 "Resistors_SMD:R_1206_HandSoldering" H 8150 3650 60  0001 C CNN
-F 3 "" H 8150 3650 60  0000 C CNN
+F 3 "http://www.vishaypg.com/docs/63070/vsmserie.pdf" H 8150 3650 60  0001 C CNN
+F 4 "Y149660R0000A0R-ND" H 8150 3650 60  0001 C CNN "Digikey/Mouser"
 	1    8150 3650
 	1    0    0    -1
@@
 F 1 "60" V 8150 4250 50  0000 C CNN
 F 2 "Resistors_SMD:R_1206_HandSoldering" H 8150 4250 60  0001 C CNN
-F 3 "" H 8150 4250 60  0000 C CNN
+F 3 "http://www.vishaypg.com/docs/63070/vsmserie.pdf" H 8150 4250 60  0001 C CNN
+F 4 "Y149660R0000A0R-ND" H 8150 4250 60  0001 C CNN "Digikey/Mouser"
 	1    8150 4250
 	1    0    0    -1

Commit message: Modifico campos de información en el esquemático para funcionar con Kicost.
Parts:
- C6: Digikey# (none) -> 311-1179-1-ND; Digikey/Mouser 311-1179-1-ND -> (none)
- J2: Digikey# (none) -> A19470-ND; Digikey/Mouser A19470-ND -> (none); Manf (none) -> AMP; Manf# (none) -> 640456-3
- R1, R2: Digikey# (none) -> CRCW120660R0KNEAIF-ND; Digikey/Mouser Y149660R0000A0R-ND -> (none); Manf (none) -> Vishay Dale; Manf# (none) -> CRCW120660R0KNEAIF
- U2: Digikey# (none) -> 766-1006-1-ND; Digikey/Mouser 766-1006-1-ND -> (none); Manf (none) -> ON; Manf# (none) -> AMIS42665TJAA1RG
- XA1: Digikey# (none) -> 952-1387-ND; Digikey/Mouser 952-1387-ND -> (none); Manf (none) -> Harwin; Manf# (none) -> M50-3502042
Changed lines of the file:
@@
 F 2 "ej2:Conn_Poncho_Derecha" H 5300 2950 60  0001 C CNN
 F 3 "https://cdn.harwin.com/pdfs/60page108.pdf" H 5300 2950 60  0001 C CNN
-F 4 "952-1387-ND" H 5300 2950 60  0001 C CNN "Digikey/Mouser"
+F 4 "Harwin" H 5300 2950 60  0001 C CNN "Manf"
+F 5 "M50-3502042" H 5300 2950 60  0001 C CNN "Manf#"
+F 6 "952-1387-ND" H 5300 2950 60  0001 C CNN "Digikey#"
 	1    5300 2950
 	1    0    0    -1
@@
 F 2 "ej2:CON_PALETA_3" H 7450 3750 60  0001 C CNN
 F 3 "http://www.te.com/commerce/DocumentDelivery/DDEController?Action=srchrtrv&DocNm=640456&DocType=Customer+Drawing&DocLang=English" H 7450 3750 60  0001 C CNN
-F 4 "A19470-ND" H 7450 3750 60  0001 C CNN "Digikey/Mouser"
+F 4 "AMP" H 7450 3750 60  0001 C CNN "Manf"
+F 5 "640456-3" H 7450 3750 60  0001 C CNN "Manf#"
+F 6 "A19470-ND" H 7450 3750 60  0001 C CNN "Digikey#"
 	1    7450 3750
 	-1   0    0    -1
@@
 F 2 "ej2:SOIC-8" H 9050 4050 60  0001 C CNN
 F 3 "http://www.onsemi.com/pub_link/Collateral/AMIS-42665-D.PDF" H 9050 4050 60  0001 C CNN
-F 4 "766-1006-1-ND" H 9050 4000 60  0001 C CNN "Digikey/Mouser"
+F 4 "ON" H 9050 4000 60  0001 C CNN "Manf"
+F 5 "AMIS42665TJAA1RG" H 9050 4000 60  0001 C CNN "Manf#"
+F 6 "766-1006-1-ND" H 9050 4000 60  0001 C CNN "Digikey#"
 	1    9050 4000
 	-1   0    0    -1
@@
 F 2 "Capacitors_SMD:C_1206_HandSoldering" H 9988 3500 30  0001 C CNN
 F 3 "http://www.yageo.com/documents/recent/UPY-GPHC_X7R_6.3V-to-50V-v12.pdf" H 9950 3650 60  0001 C CNN
-F 4 "311-1179-1-ND" H 9950 3650 60  0001 C CNN "Digikey/Mouser"
+F 4 "311-1179-1-ND" H 9950 3650 60  0001 C CNN "Digikey#"
 	1    9950 3650
 	0    1    1    0
@@
 F 2 "Resistors_SMD:R_1206_HandSoldering" H 8150 3650 60  0001 C CNN
 F 3 "http://www.vishaypg.com/docs/63070/vsmserie.pdf" H 8150 3650 60  0001 C CNN
-F 4 "Y149660R0000A0R-ND" H 8150 3650 60  0001 C CNN "Digikey/Mouser"
+F 4 "Vishay Dale" H 8150 3650 60  0001 C CNN "Manf"
+F 5 "CRCW120660R0KNEAIF" H 8150 3650 60  0001 C CNN "Manf#"
+F 6 "CRCW120660R0KNEAIF-ND" H 8150 3650 60  0001 C CNN "Digikey#"
 	1    8150 3650
 	1    0    0    -1
@@
 F 2 "Resistors_SMD:R_1206_HandSoldering" H 8150 4250 60  0001 C CNN
 F 3 "http://www.vishaypg.com/docs/63070/vsmserie.pdf" H 8150 4250 60  0001 C CNN
-F 4 "Y149660R0000A0R-ND" H 8150 4250 60  0001 C CNN "Digikey/Mouser"
+F 4 "Vishay Dale" H 8150 4250 60  0001 C CNN "Manf"
+F 5 "CRCW120660R0KNEAIF" H 8150 4250 60  0001 C CNN "Manf#"
+F 6 "CRCW120660R0KNEAIF-ND" H 8150 4250 60  0001 C CNN "Digikey#"
 	1    8150 4250
 	1    0    0    -1
