File: Ejercicio2/Rs232.sch (KiCad schematic (older format))
At the start: 7 parts, among them J1 DB9-F, U1 SP3232ECN

Commit message: Detalles visuales y agrgado de comentarios.
Other:
- moved on the sheet: J1
Changed lines of the file:
@@
 L DB9 J1
 U 1 1 564E1AB2
-P 8150 4550
-F 0 "J1" H 8150 5100 70  0000 C CNN
-F 1 "DB9-F" H 8150 4000 70  0000 C CNN
-F 2 "ej2:DB9_F_TH" H 8150 4550 60  0001 C CNN
-F 3 "http://www.sullinscorp.com/drawings/345_11773,_SDS107-PR___-_____-SN___-___.pdf" H 8150 4550 60  0001 C CNN
-F 4 "S9554-ND" H 8150 4550 60  0001 C CNN "Digikey/Mouser"
-	1    8150 4550
+P 8050 4550
+F 0 "J1" H 8050 5100 70  0000 C CNN
+F 1 "DB9-F" H 8050 4000 70  0000 C CNN
+F 2 "ej2:DB9_F_TH" H 8050 4550 60  0001 C CNN
+F 3 "http://www.sullinscorp.com/drawings/345_11773,_SDS107-PR___-_____-SN___-___.pdf" H 8050 4550 60  0001 C CNN
+F 4 "S9554-ND" H 8050 4550 60  0001 C CNN "Digikey/Mouser"
+	1    8050 4550
 	1    0    0    -1
 $EndComp
@@
 	3700 3150 4150 3150
 Wire Wire Line
-	7700 4750 6650 4750
+	7600 4750 6650 4750
 Wire Wire Line
 	6650 4750 6650 4250
@@
 	7400 4350 7400 4450
 Wire Wire Line
-	7400 4450 7700 4450
+	7400 4450 7600 4450
 Wire Wire Line
 	5750 4450 7300 4450
@@
 	7300 4450 7300 4550
 Wire Wire Line
-	7300 4550 7700 4550
+	7300 4550 7600 4550
 Wire Wire Line
 	7250 4550 7250 4650
 Wire Wire Line
-	7250 4650 7700 4650
+	7250 4650 7600 4650
 $Bitmap
 Pos 9700 3450
@@
 D7 83 7C 1A 00 80 0B F5 7C DA 77 F9 12 00 00 77 D8 F4 F5 E3 3E 81 D3 84 00 BC 9C 1F 9E 53 EF 5E
 56 13 80 F1 D0 10 7F 62 4C 03 40 06 D8 7F 03 40 06 5F ED 80 FF 91 20 12 25 DF 00 00 00 00 49 45
-4E 44 AE 42 60 82 04
+4E 44 AE 42 60 82 00
 EndData
 $EndBitmap
 Text Notes 8300 5350 2    60   ~ 0
 TIPO DCE
-NoConn ~ 7700 4250
-NoConn ~ 7700 4350
-NoConn ~ 7700 4850
-NoConn ~ 7700 4950
+NoConn ~ 7600 4250
+NoConn ~ 7600 4350
+NoConn ~ 7600 4850
+NoConn ~ 7600 4950
 $Comp
 L GND #PWR014
@@
 $EndComp
 Wire Wire Line
-	7700 4150 7450 4150
+	7600 4150 7450 4150
 Wire Wire Line
 	7450 4150 7450 4200
@@
 Text Label 3550 4350 0    60   ~ 0
 RS3
-Text HLabel 2300 3900 0    60   BiDi ~ 0
+Text HLabel 3000 3900 0    60   BiDi ~ 0
 RS[1..4]
 Wire Wire Line
@@
 	3200 4450 3300 4550
 Wire Bus Line
-	3200 4450 3200 3900
+	3200 3900 3200 4450
 Wire Bus Line
-	3200 3900 2300 3900
+	3200 3900 3000 3900
 Text Label 3550 4450 0    60   ~ 0
 RS1

Commit message: Modifico campos de información en el esquemático para funcionar con Kicost.
Parts:
- C1, C2, C4: Digikey# (none) -> 311-1179-1-ND; Digikey/Mouser 311-1179-1-ND -> (none)
- C3: Digikey/Mouser 311-1179-1-ND -> (none); digikey# (none) -> 311-1179-1-ND
- C5: Digikey# (none) -> 311-1179-1-ND; Digikey/Mouser 311-1179-1-ND -> (none); Manf (none) -> Yageo; Manf# (none) -> CC1206KRX7R9BB104
- J1: Digikey# (none) -> A35107-ND; Digikey/Mouser S9554-ND -> (none); Manf (none) -> AMP; Manf# (none) -> 1734354-1
- U1: Digikey# (none) -> 1016-1803-1-ND; Digikey/Mouser 1016-1803-1-ND -> (none); Manf (none) -> Exar; Manf# (none) -> SP3232ECN-L/TR
Changed lines of the file:
@@
 F 2 "ej2:DB9_F_TH" H 8050 4550 60  0001 C CNN
 F 3 "http://www.sullinscorp.com/drawings/345_11773,_SDS107-PR___-_____-SN___-___.pdf" H 8050 4550 60  0001 C CNN
-F 4 "S9554-ND" H 8050 4550 60  0001 C CNN "Digikey/Mouser"
+F 4 "AMP" H 8050 4550 60  0001 C CNN "Manf"
+F 5 "1734354-1" H 8050 4550 60  0001 C CNN "Manf#"
+F 6 "A35107-ND" H 8050 4550 60  0001 C CNN "Digikey#"
 	1    8050 4550
 	1    0    0    -1
@@
 F 2 "Capacitors_SMD:C_1206_HandSoldering" H 6138 3400 30  0001 C CNN
 F 3 "http://www.yageo.com/documents/recent/UPY-GPHC_X7R_6.3V-to-50V-v12.pdf" H 6100 3550 60  0001 C CNN
-F 4 "311-1179-1-ND" H 6100 3550 60  0001 C CNN "Digikey/Mouser"
+F 4 "311-1179-1-ND" H 6100 3550 60  0001 C CNN "digikey#"
 	1    6100 3550
 	0    1    1    0
@@
 F 2 "Capacitors_SMD:C_1206_HandSoldering" H 6138 3900 30  0001 C CNN
 F 3 "http://www.yageo.com/documents/recent/UPY-GPHC_X7R_6.3V-to-50V-v12.pdf" H 6100 4050 60  0001 C CNN
-F 4 "311-1179-1-ND" H 6100 4050 60  0001 C CNN "Digikey/Mouser"
+F 4 "311-1179-1-ND" H 6100 4050 60  0001 C CNN "Digikey#"
 	1    6100 4050
 	0    1    1    0
@@
 F 2 "Capacitors_SMD:C_1206_HandSoldering" H 3738 3200 30  0001 C CNN
 F 3 "http://www.yageo.com/documents/recent/UPY-GPHC_X7R_6.3V-to-50V-v12.pdf" H 3700 3350 60  0001 C CNN
-F 4 "311-1179-1-ND" H 3700 3350 60  0001 C CNN "Digikey/Mouser"
+F 4 "311-1179-1-ND" H 3700 3350 60  0001 C CNN "Digikey#"
 	1    3700 3350
 	1    0    0    -1
@@
 F 2 "Capacitors_SMD:C_1206_HandSoldering" H 3738 3700 30  0001 C CNN
 F 3 "http://www.yageo.com/documents/recent/UPY-GPHC_X7R_6.3V-to-50V-v12.pdf" H 3700 3850 60  0001 C CNN
-F 4 "311-1179-1-ND" H 3700 3850 60  0001 C CNN "Digikey/Mouser"
+F 4 "311-1179-1-ND" H 3700 3850 60  0001 C CNN "Digikey#"
 	1    3700 3850
 	1    0    0    -1
@@
 F 2 "Capacitors_SMD:C_1206_HandSoldering" H 7038 2800 30  0001 C CNN
 F 3 "http://www.yageo.com/documents/recent/UPY-GPHC_X7R_6.3V-to-50V-v12.pdf" H 7000 2950 60  0001 C CNN
-F 4 "311-1179-1-ND" H 7000 2950 60  0001 C CNN "Digikey/Mouser"
+F 4 "Yageo" H 7000 2950 60  0001 C CNN "Manf"
+F 5 "CC1206KRX7R9BB104" H 7000 2950 60  0001 C CNN "Manf#"
+F 6 "311-1179-1-ND" H 7000 2950 60  0001 C CNN "Digikey#"
 	1    7000 2950
 	1    0    0    -1
@@
 D7 83 7C 1A 00 80 0B F5 7C DA 77 F9 12 00 00 77 D8 F4 F5 E3 3E 81 D3 84 00 BC 9C 1F 9E 53 EF 5E
 56 13 80 F1 D0 10 7F 62 4C 03 40 06 D8 7F 03 40 06 5F ED 80 FF 91 20 12 25 DF 00 00 00 00 49 45
-4E 44 AE 42 60 82 01
+4E 44 AE 42 60 82 00
 EndData
 $EndBitmap
@@
 F 2 "ej2:SP3232ECN-SOIC16N" H 4950 3850 60  0001 C CNN
 F 3 "http://www.digikey.com/product-detail/es/SP3232ECN-L%2FTR/1016-1803-1-ND/3586520" H 4950 3850 60  0001 C CNN
-F 4 "1016-1803-1-ND" H 4950 3850 60  0001 C CNN "Digikey/Mouser"
+F 4 "Exar" H 4950 3850 60  0001 C CNN "Manf"
+F 5 "SP3232ECN-L/TR" H 4950 3850 60  0001 C CNN "Manf#"
+F 6 "1016-1803-1-ND" H 4950 3850 60  0001 C CNN "Digikey#"
 	1    4950 3850
 	1    0    0    -1
