File: Ejercicio2/ej2.kicad_pcb (KiCad board)
At the start: 2 copper layers, 40.6 x 61 mm, 15 parts, among them J1 DB9-F, J2 CAN, U1 SP3232ECN, U2 AMIS42665TJAA1RG

Commit message: Detalles visuales y agrgado de comentarios.
Connections:
- net /Conector/CAN_N renamed /Conector y CAN/CAN_N
- net /Conector/CAN_P renamed /Conector y CAN/CAN_P
- net /Conector/CAN_RX renamed /Conector y CAN/CAN_RX
- net /Conector/CAN_TX renamed /Conector y CAN/CAN_TX
- net /Conector/CTS renamed /Conector y CAN/CTS
- net /Conector/RTS renamed /Conector y CAN/RTS
- net /Conector/RXD renamed /Conector y CAN/RXD
- net /Conector/TXD renamed /Conector y CAN/TXD
Other:
- board text added: "Los logos se agregaron diréctamente en el PCB. Por lo tanto no están referenciados en el archivo netlist."

Commit message: Agregados de keepout, cutout areas y más textos en drawings.
Parts:
- renumbered G*** to G102
Other:
- board text added: "Cutout area (Bottom)"
- board text added: "Keepout Area (Front)"
Changed lines of the file:
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@@
     (links 44)
     (no_connects 0)
-    (area 81.072618 62.36 236.857859 164.528501)
+    (area 102.159999 73.584999 142.950001 134.695001)
     (thickness 1.6)
-    (drawings 27)
+    (drawings 36)
     (tracks 289)
     (zones 0)
@@
     (pad_to_mask_clearance 0.2)
     (aux_axis_origin 0 0)
-    (visible_elements 7FFEFFFF)
+    (visible_elements 7FFE3FFF)
     (pcbplotparams
-      (layerselection 0x00030_80000001)
+      (layerselection 0x000f0_80000001)
       (usegerberextensions false)
-      (excludeedgelayer true)
+      (excludeedgelayer false)
       (linewidth 0.100000)
       (plotframeref false)
@@
       (psa4output false)
       (plotreference true)
-      (plotvalue true)
+      (plotvalue false)
       (plotinvisibletext false)
       (padsonsilk false)
@@
       (outputformat 1)
       (mirror false)
-      (drillshape 1)
+      (drillshape 0)
       (scaleselection 1)
       (outputdirectory ""))
@@
   (module ej2:Logo_Poncho (layer F.Cu)
     (at 123.19 125.095)
-    (fp_text reference G*** (at 0.127 5.588) (layer F.SilkS) hide
-      (effects (font (thickness 0.3)))
+    (fp_text reference G102 (at 0.127 5.588) (layer F.SilkS) hide
+      (effects (font (size 0.7 0.5) (thickness 0.1)))
     )
     (fp_text value LOGO (at 0.762 7.493) (layer F.SilkS) hide
@@
       (xy 3.778435 -0.1467) (xy 3.778435 -0.1467)) (layer F.SilkS) (width 0.1))
   )
+  (gr_text "Keepout Area\n(Front)" (at 87.757 113.919) (layer Dwgs.User)
+    (effects (font (size 0.8 0.8) (thickness 0.15)) (justify right))
+  )
+  (gr_line (start 100.203 114.046) (end 99.822 114.427) (angle 90) (layer Dwgs.User) (width 0.127))
+  (gr_line (start 100.203 114.046) (end 99.822 113.665) (angle 90) (layer Dwgs.User) (width 0.127))
+  (gr_line (start 120.269 135.509) (end 119.888 136.017) (angle 90) (layer Dwgs.User) (width 0.127))
+  (gr_line (start 88.646 114.046) (end 88.773 114.046) (angle 90) (layer Dwgs.User) (width 0.127))
+  (gr_line (start 100.203 114.046) (end 88.646 114.046) (angle 90) (layer Dwgs.User) (width 0.127))
+  (gr_text "Cutout area \n(Bottom)" (at 120.523 142.367) (layer Dwgs.User)
+    (effects (font (size 0.8 0.8) (thickness 0.15)))
+  )
+  (gr_line (start 120.269 135.509) (end 120.65 136.017) (angle 90) (layer Dwgs.User) (width 0.127))
+  (gr_line (start 120.269 135.509) (end 120.269 141.605) (angle 90) (layer Dwgs.User) (width 0.127))
   (gr_line (start 158.75 123.825) (end 159.385 124.46) (angle 90) (layer Dwgs.User) (width 0.127))
   (gr_line (start 158.75 123.825) (end 159.385 123.19) (angle 90) (layer Dwgs.User) (width 0.127))
@@
     (effects (font (size 1.5 1) (thickness 0.25)))
   )
-  (gr_text "INDUSTRIA ARGENTINA" (at 115.57 132.842) (layer B.Mask)
+  (gr_text "INDUSTRIA ARGENTINA" (at 115.57 132.842) (layer B.Cu)
     (effects (font (size 1.5 1.5) (thickness 0.3)) (justify mirror))
   )
@@
     (polygon
       (pts
-        (xy 102.235 73.66) (xy 142.875 73.66) (xy 142.875 134.62) (xy 102.235 134.62)
+        (xy 142.875 134.62) (xy 102.235 134.62) (xy 102.235 73.66) (xy 142.875 73.66) (xy 142.875 134.62)
+      )
+    )
+    (polygon
+      (pts        (xy 102.997 131.445) (xy 102.997 133.985) (xy 128.397 133.985) (xy 128.397 131.445) (xy 102.997 131.445)
+      )
+    )
+  )
+  (zone (net 0) (net_name "") (layer F.Cu) (hatch edge 0.508)
+    (connect_pads (clearance 0.3048))
+    (min_thickness 0.3048)
+    (keepout (tracks allowed) (vias not_allowed) (copperpour not_allowed))
+    (fill (arc_segments 32) (thermal_gap 0.3048) (thermal_bridge_width 0.508))
+    (polygon
+      (pts
+        (xy 120.142 111.76) (xy 120.142 116.586) (xy 117.602 119.634) (xy 109.347 119.634) (xy 106.68 116.713)
+        (xy 104.14 116.713) (xy 104.14 111.76) (xy 106.68 111.76) (xy 109.22 109.22) (xy 117.602 109.22)
+        (xy 120.142 111.76)
       )
     )
@@
       )
     )
-    (polygon
-      (pts        (xy 109.22 109.22) (xy 106.68 111.76) (xy 104.14 111.76) (xy 104.14 116.713) (xy 106.68 116.713)
-        (xy 109.601 119.634) (xy 117.094 119.634) (xy 120.142 116.586) (xy 120.142 111.76) (xy 117.602 109.22)
-      )
-    )
