File: WorkshopSASE16/rele2x.kicad_pcb (KiCad board)
At the start: 2 copper layers, 85.7 x 60.3 mm, 17 parts, among them J1 TB_1X3, J2 TB_1X3, K1 RELAY_C, K2 RELAY_C, Q1 2N2222, Q2 2N2222

Commit message: Detalles al esquemático y al PCB.
Parts:
- Q1, Q2: value 2N2222 -> 2N3904
- R1, R2: value 1K -> 2K7
- R3, R4: value 220R -> 330R
Changed lines of the file:
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@@
   )
   (setup
-    (last_trace_width 0.6)
+    (last_trace_width 0.381)
     (user_trace_width 0.6)
     (user_trace_width 0.7)
@@
       (effects (font (size 1 1) (thickness 0.15)))
     )
-    (fp_text value 2N2222 (at 0 3 270) (layer F.Fab)
+    (fp_text value 2N3904 (at 0 3 270) (layer F.Fab)
       (effects (font (size 1 1) (thickness 0.15)))
     )
@@
       (effects (font (size 1 1) (thickness 0.15)))
     )
-    (fp_text value 2N2222 (at 0 3 270) (layer F.Fab)
+    (fp_text value 2N3904 (at 0 3 270) (layer F.Fab)
       (effects (font (size 1 1) (thickness 0.15)))
     )
@@
       (effects (font (size 1 1) (thickness 0.15)))
     )
-    (fp_text value 1K (at 5.08 3.81 180) (layer F.Fab)
+    (fp_text value 2K7 (at 5.08 3.81 180) (layer F.Fab)
       (effects (font (size 1 1) (thickness 0.15)))
     )
@@
       (effects (font (size 1 1) (thickness 0.15)))
     )
-    (fp_text value 1K (at 5.08 3.81 180) (layer F.Fab)
+    (fp_text value 2K7 (at 5.08 3.81 180) (layer F.Fab)
       (effects (font (size 1 1) (thickness 0.15)))
     )
@@
       (effects (font (size 1 1) (thickness 0.15)))
     )
-    (fp_text value 220R (at 5.08 3.81 180) (layer F.Fab)
+    (fp_text value 330R (at 5.08 3.81 180) (layer F.Fab)
       (effects (font (size 1 1) (thickness 0.15)))
     )
@@
       (effects (font (size 1 1) (thickness 0.15)))
     )
-    (fp_text value 220R (at 5.08 3.81 180) (layer F.Fab)
+    (fp_text value 330R (at 5.08 3.81 180) (layer F.Fab)
       (effects (font (size 1 1) (thickness 0.15)))
     )
@@
   (segment (start 141.478 86.614) (end 141.478 84.328) (width 0.6) (layer B.Cu) (net 12))
   (segment (start 140.462 87.63) (end 141.478 86.614) (width 0.6) (layer B.Cu) (net 12))
-  (segment (start 163.576 87.63) (end 165.227 87.63) (width 0.6) (layer B.Cu) (net 13) (status 400000))
-  (segment (start 165.227 83.312) (end 159.766 83.312) (width 0.6) (layer B.Cu) (net 13) (status 800000))
+  (segment (start 163.576 87.63) (end 165.227 87.63) (width 0.6) (layer B.Cu) (net 13))
+  (segment (start 165.227 83.312) (end 159.766 83.312) (width 0.6) (layer B.Cu) (net 13))
   (segment (start 166.497 84.582) (end 165.227 83.312) (width 0.6) (layer B.Cu) (net 13))
   (segment (start 166.497 86.36) (end 166.497 84.582) (width 0.6) (layer B.Cu) (net 13))
