File: WorkshopSASE16/rele2x.kicad_pcb (KiCad board)
At the start: 2 copper layers, 85.7 x 60.3 mm, 17 parts, among them J1 TB_1X3, J2 TB_1X3, K1 RELAY_C, K2 RELAY_C, Q1 2N3904, Q2 2N3904

Commit message: Corrijo error de LED invertido por biblioteca device legqacy.
Parts:
- moved LED1 2.54 mm to (140.1, 92.7), turned to 270 degrees
- moved LED2 2.54 mm to (164.2, 92.7), turned to 270 degrees
Connections:
- LED1 pad 1: +5VP -> Net-(LED1-Pad1)
- LED1 pad 2: Net-(LED1-Pad2) -> +5VP
- LED2 pad 1: +5VP -> Net-(LED2-Pad1)
- LED2 pad 2: Net-(LED2-Pad2) -> +5VP
- R3 pad 1: Net-(LED1-Pad2) -> Net-(LED1-Pad1)
- R4 pad 1: Net-(LED2-Pad2) -> Net-(LED2-Pad1)
Routing:
- net Net-(LED2-Pad2): track 4.97 -> 0.00 mm
- net Net-(LED2-Pad1): track 0.00 -> 4.97 mm
- net Net-(LED1-Pad2): track 4.97 -> 0.00 mm
- net Net-(LED1-Pad1): track 0.00 -> 4.97 mm
- net Net-(R1-Pad2): track 49.0 -> 46.5 mm
- net Net-(R2-Pad2): track 75.1 -> 76.5 mm
