File: Rele1x/rele1x.sch (KiCad schematic (older format))
At the start: 8 parts, among them J1 TB_1X3, K1 RELAY_C, Q1 2N3904

Commit message: Mejoras al ejercicio Rele1x.
Connections:
- net at K1.1: now also J1.2; no longer J1.1
- net at K1.3: now also J1.1; no longer J1.2
Changed lines of the file:
@@
 EESchema Schematic File Version 2
-LIBS:device
+LIBS:power
 LIBS:rele1x-cache
 EELAYER 25 0
@@
 Connection ~ 6900 3525
 Wire Wire Line
-	8250 4225 8100 4225
-Wire Wire Line
-	8100 4225 8100 4375
-Wire Wire Line
-	8100 4375 7550 4375
-Wire Wire Line
 	7550 4375 7550 4225
 Wire Wire Line
-	8250 3825 8250 3625
-Wire Wire Line
-	8250 3625 7500 3625
-Wire Wire Line
 	7500 3625 7500 3825
-Wire Wire Line
-	8250 4025 8100 4025
-Wire Wire Line
-	8100 4025 8100 3725
-Wire Wire Line
-	8100 3725 7600 3725
 Wire Wire Line
 	7600 3725 7600 3825
@@
 	0    1    1    0
 $EndComp
+Wire Wire Line
+	7500 3625 8150 3625
+Wire Wire Line
+	8250 3825 8150 3825
+Wire Wire Line
+	8150 3825 8150 3625
+Wire Wire Line
+	7550 4375 7950 4375
+Wire Wire Line
+	7950 4375 7950 4025
+Wire Wire Line
+	7950 4025 8250 4025
+Wire Wire Line
+	7600 3725 8050 3725
+Wire Wire Line
+	8050 3725 8050 4225
+Wire Wire Line
+	8050 4225 8250 4225
 $EndSCHEMATC

Commit message: Detalles en el PCB serigrafía, etc.
Other:
- note added: "ADVERTENCIA:\nLos componentes y sus valores se eligen\na los fines de realizar un ejercicio con KiCad.\nEn caso de querer construir el diseño, verificar \nprimero el circuito ya que este no esta verificado."
- note removed: "ADVERTENCIA:\nLos componentes y sus valores se eligen\na los fines de realizar un ejercicio con KiCad.\nEn caso de querer construir el circuito, verificar \nprimero el circuito ya que este no esta verificado."
- moved on the sheet: D1, J1, K1, LED1, Q1, R1, R2, XA1B
