File: Ejercicio1/intro.sch (KiCad schematic (older format))
At the start: 6 parts, among them K1 CONN_3

Commit message: Versión nueva del Ejercicio 1 de Kicad Tour.
Parts:
- removed R2: 100K, footprints_ej1:R3-LARGE_PADS, symbol R
- C1: footprint footprints_ej1:C_Rect_L7_W3.5_P5 -> Capacitors_THT:C_Rect_L7.0mm_W3.5mm_P5.00mm
- D1: footprint footprints_ej1:LED-3MM -> LEDs:LED_D3.0mm
- D2: footprint footprints_ej1:Diode_DO-35_SOD27_Horizontal_RM10 -> Diodes_THT:D_DO-35_SOD27_P10.16mm_Horizontal
- K1: footprint footprints_ej1:bornier3 -> Connectors:bornier3
- R1: footprint footprints_ej1:R3-LARGE_PADS -> Resistors_THT:R_Axial_DIN0204_L3.6mm_D1.6mm_P7.62mm_Horizontal
Other:
- note removed: "Resistor agregado"
Changed lines of the file:
@@
 EESchema Schematic File Version 2
+LIBS:conn
 LIBS:device
-LIBS:conn
 LIBS:intro-cache
 EELAYER 25 0
@@
 Date "2015-11-26"
 Rev "1.0"
-Comp "INTI - CMNB"
+Comp "INTI - CMNB / UNLaM  / FIUBA"
 Comment1 "Autores: Diego Brengi    Licencia:doc/LICENCIA.txt"
 Comment2 ""
@@
 F 0 "C1" H 5400 3950 50  0000 L CNN
 F 1 "100 nF" H 5400 3750 50  0000 L CNN
-F 2 "footprints_ej1:C_Rect_L7_W3.5_P5" H 5350 3850 60  0001 C CNN
+F 2 "Capacitors_THT:C_Rect_L7.0mm_W3.5mm_P5.00mm" H 5350 3850 60  0001 C CNN
 F 3 "" H 5350 3850 60  0000 C CNN
 	1    5350 3850
@@
 F 0 "R1" V 6480 4250 50  0000 C CNN
 F 1 "100K" V 6400 4250 50  0000 C CNN
-F 2 "footprints_ej1:R3-LARGE_PADS" H 6400 4250 60  0001 C CNN
+F 2 "Resistors_THT:R_Axial_DIN0204_L3.6mm_D1.6mm_P7.62mm_Horizontal" H 6400 4250 60  0001 C CNN
 F 3 "" H 6400 4250 60  0000 C CNN
 	1    6400 4250
@@
 F 0 "K1" V 4300 4200 50  0000 C CNN
 F 1 "CONN_3" V 4400 4200 40  0000 C CNN
-F 2 "footprints_ej1:bornier3" H 4350 4200 60  0001 C CNN
+F 2 "Connectors:bornier3" H 4350 4200 60  0001 C CNN
 F 3 "" H 4350 4200 60  0000 C CNN
 	1    4350 4200
@@
 Text Notes 7100 3800 0    60   Italic 0
 Resistor serie
-Wire Wire Line
-	5500 3850 6700 3850
-Wire Wire Line
-	5500 4700 6700 4700
 $Comp
 L LED D1
@@
 F 0 "D1" H 5350 3650 50  0000 C CNN
 F 1 "LED ROJO 5mm" H 5350 3400 50  0000 C CNN
-F 2 "footprints_ej1:LED-3MM" H 5350 3550 60  0001 C CNN
+F 2 "LEDs:LED_D3.0mm" H 5350 3550 60  0001 C CNN
 F 3 "" H 5350 3550 60  0000 C CNN
 	1    5350 3550
@@
 F 0 "D2" H 5350 4800 40  0000 C CNN
 F 1 "1N4148" H 5350 4600 40  0000 C CNN
-F 2 "footprints_ej1:Diode_DO-35_SOD27_Horizontal_RM10" H 5350 4700 60  0001 C CNN
+F 2 "Diodes_THT:D_DO-35_SOD27_P10.16mm_Horizontal" H 5350 4700 60  0001 C CNN
 F 3 "" H 5350 4700 60  0000 C CNN
 	1    5350 4700
 	1    0    0    -1
 $EndComp
-$Comp
-L R R2
-U 1 1 564A3B91
-P 6700 4250
-F 0 "R2" V 6780 4250 50  0000 C CNN
-F 1 "100K" V 6700 4250 50  0000 C CNN
-F 2 "footprints_ej1:R3-LARGE_PADS" V 6630 4250 30  0001 C CNN
-F 3 "" H 6700 4250 30  0000 C CNN
-	1    6700 4250
-	1    0    0    -1
-$EndComp
 Wire Wire Line
-	6700 3850 6700 4100
-Connection ~ 6400 3850
+	5500 3850 6400 3850
 Wire Wire Line
-	6700 4700 6700 4400
-Connection ~ 6400 4700
-Wire Notes Line
-	6800 4150 7000 3950
-Wire Notes Line
-	7000 3950 7200 3950
-Text Notes 7250 4000 0    60   ~ 0
-Resistor agregado
+	6400 4700 5500 4700
 $EndSCHEMATC
