File: oscilador-multicapa/Oscilador_1.sch (KiCad schematic (older format))
At the start: 4 parts

Commit message: Ejercicio terminado multicapa.
Parts:
- added F1, F2: Fiducial, Fiducial:Fiducial_1mm_Dia_2mm_Outer, symbol Mechanical:MountingHole
- MK101, MK102, MK103, MK104: symbol Oscilador_1-rescue:Mounting_Hole -> resc:Mounting_Hole
Changed lines of the file:
@@
 encoding utf-8
 Sheet 1 3
-Title "OSCILIADOR CON 40106 Y DOS LEDS - PRINCIPAL"
-Date "2018-06-16"
+Title "OSCILIADOR CON 40106 Y DOS LEDS"
+Date "2018-09-28"
 Rev "1.0"
-Comp "Taller de Electrónica - UNLaM"
+Comp "Curso KiCad Multicapa"
 Comment1 "Autor: Diego Brengi"
 Comment2 ""
@@
 	5550 3550 6150 3550
 $Comp
-L Oscilador_1-rescue:Mounting_Hole MK101
+L resc:Mounting_Hole MK101
 U 1 1 5B340FE4
 P 4700 4950
@@
 $EndComp
 $Comp
-L Oscilador_1-rescue:Mounting_Hole MK102
+L resc:Mounting_Hole MK102
 U 1 1 5B3410A9
 P 4700 5300
@@
 $EndComp
 $Comp
-L Oscilador_1-rescue:Mounting_Hole MK103
+L resc:Mounting_Hole MK103
 U 1 1 5B3410EE
 P 5450 4950
@@
 $EndComp
 $Comp
-L Oscilador_1-rescue:Mounting_Hole MK104
+L resc:Mounting_Hole MK104
 U 1 1 5B34113B
 P 5450 5300
@@
 	1    0    0    -1
 $EndComp
+$Comp
+L Mechanical:MountingHole F1
+U 1 1 5BAC17FD
+P 6275 4925
+F 0 "F1" H 6375 4971 50  0000 L CNN
+F 1 "Fiducial" H 6375 4880 50  0000 L CNN
+F 2 "Fiducial:Fiducial_1mm_Dia_2mm_Outer" H 6275 4925 50  0001 C CNN
+F 3 "~" H 6275 4925 50  0001 C CNN
+	1    6275 4925
+	1    0    0    -1
+$EndComp
+$Comp
+L Mechanical:MountingHole F2
+U 1 1 5BAE4FFF
+P 6275 5300
+F 0 "F2" H 6375 5346 50  0000 L CNN
+F 1 "Fiducial" H 6375 5255 50  0000 L CNN
+F 2 "Fiducial:Fiducial_1mm_Dia_2mm_Outer" H 6275 5300 50  0001 C CNN
+F 3 "~" H 6275 5300 50  0001 C CNN
+	1    6275 5300
+	1    0    0    -1
+$EndComp
