File: oscilador-multicapa/leds.sch (KiCad schematic (older format))
At the start: 8 parts, among them Q301 BC546, Q302 BC546

Commit message: Ejercicio terminado multicapa.
Parts:
- D301, D302: symbol Oscilador_1-rescue:LED -> resc:LED
- Q301, Q302: symbol Oscilador_1-rescue:BC546 -> resc:BC546
- R301, R302, R303, R304: symbol Oscilador_1-rescue:R -> resc:R
Changed lines of the file:
@@
 encoding utf-8
 Sheet 3 3
-Title "OSCILIADOR CON 40106 Y DOS LEDS - LEDS INDICADORES"
-Date "2018-06-16"
-Rev ""
-Comp "Taller de Electrónica - UNLaM"
+Title "OSCILIADOR CON 40106 Y DOS LEDS"
+Date "2018-09-28"
+Rev "1.0"
+Comp "Curso KiCad Multicapa"
 Comment1 "Autor: Diego Brengi"
 Comment2 ""
@@
 $EndDescr
 $Comp
-L Oscilador_1-rescue:R R302
+L resc:R R302
 U 1 1 5B294EA7
 P 5050 2900
@@
 $EndComp
 $Comp
-L Oscilador_1-rescue:R R303
+L resc:R R303
 U 1 1 5B294EAE
 P 5800 3650
@@
 $EndComp
 $Comp
-L Oscilador_1-rescue:R R301
+L resc:R R301
 U 1 1 5B294EB5
 P 4350 3650
@@
 $EndComp
 $Comp
-L Oscilador_1-rescue:LED D301
+L resc:LED D301
 U 1 1 5B294EBC
 P 5050 3250
@@
 $EndComp
 $Comp
-L Oscilador_1-rescue:BC546 Q301
+L resc:BC546 Q301
 U 1 1 5B294EC3
 P 4950 3650
@@
 	6350 2700 6350 2750
 $Comp
-L Oscilador_1-rescue:R R304
+L resc:R R304
 U 1 1 5B294EE3
 P 6350 2900
@@
 $EndComp
 $Comp
-L Oscilador_1-rescue:LED D302
+L resc:LED D302
 U 1 1 5B294EEA
 P 6350 3250
@@
 	6350 3850 6350 3900
 $Comp
-L Oscilador_1-rescue:BC546 Q302
+L resc:BC546 Q302
 U 1 1 5B294EF8
 P 6250 3650
