File: oscilador-multicapa/oscilador.sch (KiCad schematic (older format))
At the start: 8 parts, among them J201 Conn_01x02, U201 40106

Commit message: Ejercicio terminado multicapa.
Parts:
- C201: symbol Oscilador_1-rescue:CP -> resc:CP
- C202: symbol Oscilador_1-rescue:C -> resc:C
- D201, D202: symbol Oscilador_1-rescue:D -> resc:D
- J201: symbol Oscilador_1-rescue:CONN_01X02 -> resc:CONN_01X02
- R201, R202: symbol Oscilador_1-rescue:R -> resc:R
- U201: symbol Oscilador_1-rescue:40106 -> resc:40106
Connections:
- wire segments 29 -> 38
Changed lines of the file:
@@
 encoding utf-8
 Sheet 2 3
-Title "OSCILIADOR CON 40106 Y DOS LEDS - OSCILADOR"
-Date "2018-06-16"
-Rev ""
-Comp "Taller de Electrónica - UNLaM"
+Title "OSCILIADOR CON 40106 Y DOS LEDS"
+Date "2018-09-28"
+Rev "1.0"
+Comp "Curso KiCad Multicapa"
 Comment1 "Autor: Diego Brengi"
 Comment2 ""
@@
 $EndComp
 $Comp
-L Oscilador_1-rescue:40106 U201
+L resc:40106 U201
 U 1 1 5B295443
 P 4850 3550
@@
 $EndComp
 $Comp
-L Oscilador_1-rescue:40106 U201
+L resc:40106 U201
 U 2 1 5B29544A
 P 4900 5500
@@
 $EndComp
 $Comp
-L Oscilador_1-rescue:40106 U201
+L resc:40106 U201
 U 3 1 5B295451
 P 6200 5500
@@
 $EndComp
 $Comp
-L Oscilador_1-rescue:C C202
+L resc:C C202
 U 1 1 5B295458
 P 5250 2750
@@
 $EndComp
 $Comp
-L Oscilador_1-rescue:CP C201
+L resc:CP C201
 U 1 1 5B29545F
 P 4350 4550
@@
 $EndComp
 $Comp
-L Oscilador_1-rescue:R R201
+L resc:R R201
 U 1 1 5B295466
 P 4850 4050
@@
 $EndComp
 $Comp
-L Oscilador_1-rescue:R R202
+L resc:R R202
 U 1 1 5B29546D
 P 4850 4450
@@
 $EndComp
 $Comp
-L Oscilador_1-rescue:D D201
+L resc:D D201
 U 1 1 5B295474
 P 5300 4050
@@
 $EndComp
 $Comp
-L Oscilador_1-rescue:D D202
+L resc:D D202
 U 1 1 5B29547B
 P 5300 4450
@@
 $EndComp
 $Comp
-L Oscilador_1-rescue:CONN_01X02 J201
+L resc:CONN_01X02 J201
 U 1 1 5B295482
 P 4350 2750
@@
 	4700 4050 4600 4050
 Wire Wire Line
-	4600 4050 4600 4450
+	4600 4050 4600 4250
 Wire Wire Line
 	4600 4450 4700 4450
@@
 	5000 4450 5150 4450
 Wire Wire Line
-	5350 3550 5700 3550
+	5350 3550 5600 3550
 Wire Wire Line
 	5600 4450 5450 4450
 Wire Wire Line
-	5600 3550 5600 4450
+	5600 3550 5600 4050
 Connection ~ 5600 3550
 Wire Wire Line
@@
 	4350 4750 4350 4700
 Wire Wire Line
-	4350 3550 4350 4400
+	4350 3550 4350 4250
 Wire Wire Line
 	5250 2600 5000 2600
@@
 	5000 2600 5000 2700
 Wire Wire Line
-	5000 2700 4550 2700
+	5000 2700 4850 2700
 Wire Wire Line
 	5250 2900 5000 2900
@@
 	5000 2900 5000 2800
 Wire Wire Line
-	5000 2800 4550 2800
+	5000 2800 4850 2800
 Wire Wire Line
 	4850 2950 4850 2800
@@
 	6700 5500 6800 5500
 Wire Wire Line
-	5400 5500 5700 5500
+	5400 5500 5550 5500
 Wire Wire Line
 	5550 5500 5550 4950
@@
 Text Label 4350 5500 2    60   ~ 0
 OSC
+Wire Wire Line
+	4350 4250 4350 4400
+Wire Wire Line
+	4600 4250 4600 4450
+Wire Wire Line
+	5600 3550 5700 3550
+Wire Wire Line
+	5600 4050 5600 4450
+Wire Wire Line
+	4850 2800 4600 2800
+Wire Wire Line
+	4850 2700 4600 2700
+Wire Wire Line
+	5550 5500 5700 5500
+Wire Wire Line
+	4600 2700 4550 2700
+Wire Wire Line
+	4600 2800 4550 2800
 $EndSCHEMATC
