File: tourk6/tourk6.kicad_sch (KiCad schematic)
At the start: 5 parts, among them J1 Conn_01x03

Commit message: Avances en el PCB.
Parts:
- D2: footprint Diode_THT:D_A-405_P7.62mm_Horizontal -> Diode_THT:D_DO-34_SOD68_P7.62mm_Horizontal
Changed lines of the file:
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@@
     (property "Reference" "D2" (id 0) (at 99.06 74.93 0))
     (property "Value" "1n4148" (id 1) (at 99.06 77.47 0))
-    (property "Footprint" "Diode_THT:D_A-405_P7.62mm_Horizontal" (id 2) (at 99.06 81.28 0)
+    (property "Footprint" "Diode_THT:D_DO-34_SOD68_P7.62mm_Horizontal" (id 2) (at 99.06 81.28 0)
       (effects (font (size 1.27 1.27)) hide)
     )
@@
     )
     (path "/ada24e41-1fbe-46a1-b443-9a8a24faea53"
-      (reference "D2") (unit 1) (value "1n4148") (footprint "Diode_THT:D_A-405_P7.62mm_Horizontal")
+      (reference "D2") (unit 1) (value "1n4148") (footprint "Diode_THT:D_DO-34_SOD68_P7.62mm_Horizontal")
     )
     (path "/c7e61b09-b828-49fa-9de0-37f5b6077b27"
